Commit message: Update comment and readme

File: resources/robots/g1_description/g1_15dof.urdf (robot description, URDF)
Before this commit: robot g1_15dof, 39 links, 38 joints
Links:
- link waist_yaw_link: mass 0.214 -> 0.244; geometry visual mesh filename=meshes/waist_yaw_link.STL
Joints:
- joint waist_yaw_joint: type fixed -> revolute
